File: hardware/NullWiiCon v2/NullWiiCon v2.kicad_pcb (KiCad board)
At the start: 2 copper layers, 71.2 x 22.6 mm, 54 parts, among them J1 USB_C_Receptacle_USB2.0, J2 Conn_01x05_Female, J4 Conn_01x05_Female, J5 Conn_02x03_Odd_Even, J6 Conn_01x03_Female, P1 CONN_WII, SW1 SW_Push, SW2 SW_DIP_x05, U1 MCP1700-3302E_SOT23, U2 ATmega32U4-MU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

Commit message: Start of PCB 2.1
Parts:
- removed the G*** at (102.6, 119.8)
- added D4: STATUS, LED_SMD:LED_0603_1608Metric, F.Cu at (109.3, 102.8)
- added G***: LOGO, Logos:NullWiiCon v2.1, F.Cu at (103.3, 119.9)
- added R13: 10k, Resistor_SMD:R_0402_1005Metric, F.Cu at (109.3, 105.8)
- moved D1 2.33 mm to (107.0, 102.8)
- moved R3 2.33 mm to (107.0, 105.8)
- moved D2 1.23 mm to (104.7, 102.8)
- moved R5 1.23 mm to (104.7, 105.8)
- renumbered Ce to C8
Connections:
- C10 pad 1: +5V -> +3V3
- C9 pad 1: +5V -> +3V3
- J6 pad 2: +5V -> +3V3
- JP9 pad 2: +5V -> +3V3
- U2 pad 32: /DIP_SW1 -> /STATUS
- U2 pad 41: Net-(U2-Pad41) -> /DIP_SW1
- U3 pad 3: Net-(U3-Pad3) -> Net-(JP7-Pad2)
- U3 pad 8: +5V -> +3V3
- U4 pad 3: Net-(U4-Pad3) -> Net-(JP1-Pad1)
- U4 pad 8: +5V -> +3V3
Routing:
- net +3V3: track 68.1 -> 113.6 mm, vias 0 -> 3
- net +5V: track 156.4 -> 133.3 mm
- net /STATUS: track 0.00 -> 13.8 mm
- net GND: track 47.6 -> 43.3 mm, vias 16 -> 17
- net /DIP_SW1: track 27.1 -> 23.3 mm
- net /TX_LED: track 32.1 -> 34.3 mm
- net /S: track 76.7 -> 74.8 mm
- net Net-(D4-Pad1): track 0.00 -> 1.69 mm
- net /SCL: track 96.3 -> 98.0 mm
- net Net-(JP7-Pad2): track 4.45 -> 5.72 mm
- net Net-(JP1-Pad1): track 5.54 -> 6.81 mm
- net /WP: track 11.5 -> 12.4 mm
- net /RX_LED: track 20.1 -> 20.7 mm

Commit message: PCB V2.1
Parts:
- C1, C10, C2, C3, C4, C5, C6, C7, C8, C9: footprint Capacitor_SMD:C_0402_1005Metric -> DIP:C_0402_1005Metric
- R1, R10, R11, R12, R13, R2, R3, R4, R5, R6, R7, R8, R9: footprint Resistor_SMD:R_0402_1005Metric -> DIP:R_0402_1005Metric
