File: hardware/NullWiiCon v2_Slim/NullWiiCon v2_Slim.kicad_pcb (KiCad board)
At the start: 2 copper layers, 43.9 x 27.3 mm, 46 parts, among them J1 USB_C_Receptacle_USB2.0, J2 Conn_01x05_Female, J4 Conn_01x05_Female, J5 Conn_02x03_Odd_Even, J6 Conn_01x03_Female, P1 CONN_WII, SW1 SW_Push, U1 MCP1700-3302E_SOT23, U2 ATmega32U4-MU, U3 CAT24C256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

Commit message: PCB V2.1
Parts:
- added REF**: KiCad-Logo_5mm_SilkScreen, Symbol:KiCad-Logo_5mm_SilkScreen, B.Cu at (95.6, 103.0)
- C1, C10, C2, C3, C4, C5, C6, C7, C8, C9: footprint Capacitor_SMD:C_0402_1005Metric -> DIP:C_0402_1005Metric
- Logo1: footprint Logos:NullWiiCon v2 -> Logos:NullWiiCon v2.1
- R1, R10, R11, R12, R13, R14, R2, R3, R4, R5, R6, R7, R8, R9: footprint Resistor_SMD:R_0402_1005Metric -> DIP:R_0402_1005Metric
- U2: footprint Package_DFN_QFN:QFN-44-1EP_7x7mm_P0.5mm_EP5.2x5.2mm -> DIP:QFN-44-1EP_7x7mm_P0.5mm_EP5.2x5.2mm_no_midpaste_smaller_EP
- moved Logo1 0.89 mm to (85.0, 95.1)
- moved C7 0.51 mm to (92.3, 99.5)
Connections:
- C10 pad 1: +5V -> +3V3
- C9 pad 1: +5V -> +3V3
- J6 pad 2: +5V -> +3V3
- JP9 pad 2: +5V -> +3V3
- U3 pad 3: Net-(U3-Pad3) -> Net-(JP7-Pad2)
- U3 pad 8: +5V -> +3V3
- U4 pad 3: Net-(U4-Pad3) -> Net-(JP1-Pad1)
- U4 pad 8: +5V -> +3V3
Routing:
- net +3V3: track 34.3 -> 67.7 mm, vias 0 -> 3
- net +5V: track 147.8 -> 116.2 mm, vias 4 -> 2
- net Net-(JP7-Pad2): track 3.98 -> 5.25 mm
- net Net-(JP1-Pad1): track 3.11 -> 4.38 mm
- net GND: track 41.6 -> 42.5 mm, vias 18 -> 20
- net Net-(C7-Pad1): track 1.90 -> 2.41 mm
